File: KiCad/fireball_fc/fireball_fc.kicad_sch (KiCad schematic)
At the start: 0 parts

Commit message: let's go
Parts:
- added C5: 4.7uF, Capacitor_SMD:C_0805_2012Metric, symbol Device:C_Small
- added C6, C8: 0.1uF, Capacitor_SMD:C_0402_1005Metric, symbol Device:C_Small
- added C7: 1uF, Capacitor_SMD:C_0805_2012Metric, symbol Device:C_Small
- added D1: D, Capacitor_SMD:C_0805_2012Metric, symbol Device:D
- added D2: BZV55B5V1, Diode_SMD:D_MiniMELF, symbol Diode:BZV55B5V1
- added D4: LED, LED_SMD:LED_0805_2012Metric, symbol Device:LED
- added D5: WS2812B-2020, LED_SMD:LED_WS2812B-2020_PLCC4_2.0x2.0mm, symbol LED:WS2812B-2020
- added J1: Micro_SD_Card, Connector_Card:microSD_HC_Hirose_DM3BT-DSF-PEJS, symbol Connector:Micro_SD_Card
- added J3: Conn_01x04, Connector_PinSocket_2.54mm:PinSocket_1x04_P2.54mm_Vertical, symbol Connector_Generic:Conn_01x04
- added J4: Conn_01x03, Connector_PinSocket_2.54mm:PinSocket_1x03_P2.54mm_Vertical, symbol Connector_Generic:Conn_01x03
- added J6: Conn_01x02, Connector_PinSocket_2.54mm:PinSocket_1x02_P2.54mm_Vertical, symbol Connector_Generic:Conn_01x02
- added P1: USB_C_Plug_USB2.0, Connector_USB:USB_C_Receptacle_GCT_USB4105-xx-A_16P_TopMnt_Horizontal, symbol Connector:USB_C_Plug_USB2.0
- added R1: R_Small, symbol Device:R_Small
- added U1: RP2040, Package_DFN_QFN:QFN-56-1EP_7x7mm_P0.4mm_EP3.2x3.2mm, symbol MCU_RaspberryPi:RP2040
- added U2: MAX17048G, symbol fireball:MAX17048G
- added U3: MS5607-02BA, Package_LGA:LGA-8_3x5mm_P1.25mm, symbol Sensor_Pressure:MS5607-02BA
- added U4: TPS61023, Package_TO_SOT_SMD:SOT-563, symbol fireball:TPS61023
- added U5: LSM6DSO, Package_LGA:LGA-14_3x2.5mm_P0.5mm_LayoutBorder3x4y, symbol fireball:LSM6DSO
- added U6: NCP708, Package_DFN_QFN:DFN-6-1EP_3x3mm_P0.95mm_EP1.7x2.6mm, symbol symbols:NCP708-3v3
Connections:
- new net: P1.A1 (GND), P1.A12 (GND), P1.B1 (GND), P1.B12 (GND)
- new net: P1.A4 (VBUS), P1.A9 (VBUS), P1.B4 (VBUS), P1.B9 (VBUS)
- new net: U3.4 (CSB), U3.5 (CSB)
- new net: D4.1 (K), R1.2
- new net: U1.1 (IOVDD), U1.10 (IOVDD), U1.22 (IOVDD), U1.33 (IOVDD), U1.42 (IOVDD), U1.49 (IOVDD)
- new net: U1.23 (DVDD), U1.50 (DVDD)
- new net +3V3: C5.1, C6.2, D2.1 (K), D4.2 (A), J3.2 (Pin_2), U6.4 (OUT), U6.5 (OUT_S)
- new net +5V: C7.1, C8.2, D1.1 (K), U6.1 (EN), U6.6 (IN)
- new net +BATT: D1.2 (A), J4.2 (Pin_2), J6.2 (Pin_2)
- new net GND: C5.2, C6.1, C7.2, C8.1, D2.2 (A), J3.1 (Pin_1), J4.1 (Pin_1), J6.1 (Pin_1), R1.1, U6.2 (GND), U6.3 (N/C), U6.7 (PAD)
- new net GPS_RX: J3.3 (Pin_3)
- new net GPS_TX: J3.4 (Pin_4)
- new net VTX: J4.3 (Pin_3)
- no-connect marks 0 -> 3
Other:
- note added: "Barometer"
- note added: "Battery Input"
- note added: "Boost"
- note added: "GPS"
- note added: "IMU"
- note added: "LiPo Fuel"
- note added: "NeoPixel"
- note added: "Power LED"
- note added: "SD"
- note added: "USB"
- note added: "USB Voltage Regulator Circuit"
- note added: "VTX"
