File: KiCad/fireball_fc/fireball_fc.kicad_sch (KiCad schematic)
At the start: 20 parts, among them J1 Micro_SD_Card, J3 Conn_01x04, J4 Conn_01x03, J6 Conn_01x02, P1 USB_C_Plug_USB2.0, U1 RP2040, U2 MAX17048G, U3 MS5607-02BA, U4 TPS61023, U5 LSM6DSO, U6 NCP708

Commit message: add baro and lipo fuel hookups
Parts:
- added BZ1: Buzzer, symbol Device:Buzzer
- added C1: C_Small, symbol Device:C_Small
- added C3, C4: 0.1uF, Capacitor_SMD:C_0402_1005Metric, symbol Device:C_Small
Connections:
- net +3V3: now also U3.1 (VDD), U3.2 (PS), C3.2, C4.2
- net +BATT: now also U2.2 (CELL), U2.3 (VDD), C1.2
- net GND: now also U2.1 (CTG), U2.4 (GND), U2.6 (Q), U2.9 (PAD), U3.3 (GND), BZ1.2 (-), C1.1, C3.1, C4.1
- net SDA: now reaches U3.7 (SDI/SDA)
- net SDA: now also U2.8 (SDA)
- net SCL: now reaches U3.8 (SCLK)
- net SCL: now also U2.7 (SCL)
Other:
- note added: "Buzzer"
- moved on the sheet: U2, U5

Commit message: largely finished my portion
Parts:
- removed J4: Conn_01x03, Connector_PinSocket_2.54mm:PinSocket_1x03_P2.54mm_Vertical, symbol Connector_Generic:Conn_01x03
- added C10, C9: 0.1uF, Capacitor_SMD:C_0402_1005Metric, symbol Device:C_Small
- added C11, C12: 22uF, symbol Device:C_Small
- added C2: 10uF, symbol Device:C_Small
- added L1: 1uH (1 ohm), symbol Device:L_Small
- added R2: 732k, symbol Device:R_Small
- added R3: 100k, symbol Device:R_Small
- C1: value C_Small -> 0.1uF
Connections:
- net +3V3: now also U5.5 (VDDIO), U5.8 (VDD), C10.1, C9.1
- net +5V: now also U4.1 (FB), C11.2, C12.2, R2.2, R3.2
- net +BATT: now also U4.3 (VIN), C2.2, L1.1
- net GND: now also U4.4 (GND), U5.1 (SDO/SA0), U5.2 (SDX), U5.3 (SCX), U5.6 (GND), U5.7 (GND), C10.2, C11.1, C12.1, C2.1, C9.2, R3.1
- net SCL: now also U5.13 (SCL)
- net SDA: now also U5.14 (SDA)
- net 5V_EN: now reaches U4.2 (EN)
- net at U4.5 (SW): now also L1.2
- net at U4.6 (VOUT): now also R2.1
- no-connect marks 3 -> 8
Other:
- note added: "Batt Plug"
- note removed: "Battery Input"
- note removed: "VTX"
- moved on the sheet: C7, C8, D5, J3, J6, P1, U2, U4, U5

Commit message: Done for now
Parts:
- removed J1: Micro_SD_Card, Connector_Card:microSD_HC_Hirose_DM3BT-DSF-PEJS, symbol Connector:Micro_SD_Card
- added C13, C15, C16, C19, C20: 0.1uF, symbol Device:C_Small
- added C14: 1uF, symbol Device:C_Small
- added C17, C18: 15pF, symbol Device:C_Small
- added CN1: HDGC2001WR-S-4P, lcsc_footprints:C2936226_CONN-SMD_4P-P2_00_HDGC_HDGC2001WR-S-4P, symbol lcsc_imported:HDGC2001WR-S-4P
- added CN2: HDGC2001WR-S-3P, lcsc_footprints:C2936225_CONN-SMD_3P-P2_00_HDGC_HDGC2001WR-S-3P, symbol lcsc_imported:HDGC2001WR-S-3P
- added Card1: HYC77-TF09-200, lcsc_footprints:C341092_TF-SMD_HYC77-TF09-200, symbol lcsc_imported:HYC77-TF09-200
- added D6: LED, LED_SMD:LED_0805_2012Metric, symbol Device:LED
- added D7, D8, D9: WS2812B-2020, LED_SMD:LED_WS2812B-2020_PLCC4_2.0x2.0mm, symbol LED:WS2812B-2020
- added R4: 220ohm, Resistor_SMD:R_0402_1005Metric, symbol Device:R_Small
- added R5: 5.1k, symbol Device:R_Small
- added SW1: HX 3X4X2-2P-2.5N-04, lcsc_footprints:C54407262_SW-SMD_L4_0-W3_0-LS5_0, symbol lcsc_imported:HX_3X4X2-2P-2_5N-04
- added U7: W25Q128JVS, Package_SO:SOIC-8_5.3x5.3mm_P1.27mm, symbol Memory_Flash:W25Q128JVS
- added U8: W25Q16JVUXIQ, lcsc_footprints:C2843335_USON-8_L3_0-W2_0-P0_50-BL-EP, symbol lcsc_imported:W25Q16JVUXIQ
- added U9: HDGC2001WR-S-9P, lcsc_footprints:C5175304_CONN-SMD_9P-P2_00_HDGC_HDGC2001WR-S-9P, symbol lcsc_imported:HDGC2001WR-S-9P
- added X2: 12MHZ Crystal, lcsc_footprints:C157341_OSC-SMD_4P-L5_0-W3_2-BL, symbol lcsc_imported:X50328MSB4SI
- R1: value R_Small -> 220ohm; footprint (none) -> Resistor_SMD:R_0402_1005Metric
Connections:
- net +3V3: now also D5.4 (VDD), U1.1 (IOVDD), U1.10 (IOVDD), U1.22 (IOVDD), U1.33 (IOVDD), U1.42 (IOVDD), U1.43 (ADC_AVDD), U1.44 (VREG_VIN), U1.48 (USB_VDD), U1.49 (IOVDD), C13.2, C15.2, C16.1, C19.1, C20.1, D7.4 (VDD), D8.4 (VDD), D9.4 (VDD), U7.8 (VCC), U8.8 (VCC)
- net +5V: now also P1.A4 (VBUS), P1.A9 (VBUS), P1.B4 (VBUS), P1.B9 (VBUS), CN2.2
- net GND: now also D5.2 (VSS), P1.A1 (GND), P1.A12 (GND), P1.B1 (GND), P1.B12 (GND), P1.SH (SHIELD), U1.19 (TESTEN), U1.57 (GND), C13.1, C14.1, C15.1, C16.2, C17.2, C18.2, C19.2, C20.2, CN1.4, CN1.5, CN1.6, CN2.3, CN2.4, CN2.5, Card1.10, Card1.11, Card1.12, Card1.13, D7.2 (VSS), D8.2 (VSS), D9.2 (VSS), R4.1, R5.1, U7.4 (GND), U8.4 (GND), U8.9 (EP), U9.10, U9.11, U9.8, X2.2 (GND), X2.4 (GND)
- net GPS_RX: now also CN1.1; no longer J3.3 (Pin_3)
- net GPS_TX: now also CN1.2; no longer J3.4 (Pin_4)
- net at P1.A5 (CC): now also R5.2
- net USBDATA+: now reaches P1.A6 (D+)
- net USBDATA+: now also U1.47 (USB_DP)
- net USBDATA-: now reaches P1.A7 (D-)
- net USBDATA-: now also U1.46 (USB_DM)
- net at D5.3 (DIN): now also D7.1 (DOUT)
- net at U1.20 (XIN): now also C17.1, X2.1 (OSC1)
- net at U1.21 (XOUT): now also C18.1, X2.3 (OSC2)
- net at U1.24 (SWCLK): now also J3.4 (Pin_4)
- net at U1.25 (SWDIO): now also J3.3 (Pin_3)
- net at U1.45 (VREG_VOUT): now also C14.2
- net at U1.51 (QSPI_SD3): now also U8.7 (HOLD#orRESET#(IO3))
- net at U1.52 (QSPI_SCLK): now also U8.6 (CLK)
- net at U1.53 (QSPI_SD0): now also U8.5 (DI(IO0))
- net at U1.54 (QSPI_SD2): now also U8.3 (WP#(IO2))
- net at U1.55 (QSPI_SD1): now also U8.2 (DO(IO1))
- net at U1.56 (~{QSPI_SS}): now also U8.1 (CS#)
- new net: D6.1 (K), R4.2
- new net: D7.3 (DIN), D8.1 (DOUT)
- new net: D8.3 (DIN), D9.1 (DOUT)
- new net 3.3V: CN1.3, U9.9
- new net DVR: CN2.1
- new net FLASH_CLK: U7.6 (CLK)
- new net FLASH_CS: U7.1 (~{CS})
- new net FLASH_IO0: U7.5 (DI/IO_{0})
- new net FLASH_IO1: U7.2 (DO/IO_{1})
- new net FLASH_IO2: U7.3 (~{WP}/IO_{2})
- new net FLASH_IO3: U7.7 (~{HOLD}/~{RESET}/IO_{3})
- new net LORA_CS: U9.2
- new net LORA_DIO0: U9.6
- new net LORA_EN: U9.7
- new net LORA_MISO: U9.4
- new net LORA_MOSI: U9.3
- new net LORA_RST: U9.1
- new net LORA_SCK: U9.5
- new net NEOPIXEL: D9.3 (DIN)
- new net SDLED: D6.2 (A)
- no-connect marks 8 -> 10
Other:
- note added: "Breathing effect when writing, solid when idle, blink when error"
- note added: "DVR + accessory power"
- note added: "LORA Connector"
- note added: "MCU + Flash(code)"
- note added: "SD Status LED"
- note added: "Storage Flash"
- note added: "use the one that I just imported"
- note added: "we need to define which led means what. we can encode messages in light patterns."
- moved on the sheet: BZ1, C11, C12, C2, J3, L1, R2, R3, U1, U4

Commit message: more schematic
Parts:
- removed C16: 0.1uF, symbol Device:C_Small
- removed C17: 15pF, symbol Device:C_Small
- removed U7: W25Q128JVS, Package_SO:SOIC-8_5.3x5.3mm_P1.27mm, symbol Memory_Flash:W25Q128JVS
- removed U8: W25Q16JVUXIQ, lcsc_footprints:C2843335_USON-8_L3_0-W2_0-P0_50-BL-EP, symbol lcsc_imported:W25Q16JVUXIQ
- added C1: 15pF, Capacitor_SMD:C_0402_1005Metric, symbol Device:C_Small
- added C19: 0.1uF, Capacitor_SMD:C_0402_1005Metric, symbol Device:C_Small
- added SW2: MAIN POWER, Connector_PinSocket_2.54mm:PinSocket_1x02_P2.54mm_Vertical, symbol Switch:SW_SPST
- added U4: CAT24C256WI-GT3, Package_SO:SOIC-8-1EP_3.9x4.9mm_P1.27mm_EP2.29x3mm, symbol fireball:MB85RC256VPF
- added U7: W25Q16JVUXIQ, lcsc_footprints:C2843335_USON-8_L3_0-W2_0-P0_50-BL-EP, symbol lcsc_imported:W25Q16JVUXIQ
- BZ1: footprint (none) -> Buzzer_Beeper:Buzzer_CUI_CPT-9019S-SMT
- C10: renamed from C12; footprint (none) -> Capacitor_SMD:C_0805_2012Metric
- C12: renamed from C15; footprint (none) -> Capacitor_SMD:C_0402_1005Metric
- C2: renamed from C18; footprint (none) -> Capacitor_SMD:C_0402_1005Metric
- C3: renamed from C20; footprint (none) -> Capacitor_SMD:C_0402_1005Metric
- C4: renamed from C19; footprint (none) -> Capacitor_SMD:C_0402_1005Metric
- C5: renamed from C13; footprint (none) -> Capacitor_SMD:C_0402_1005Metric
- C6: renamed from C14; footprint (none) -> Capacitor_SMD:C_0603_1608Metric
- C7: renamed from C1; footprint (none) -> Capacitor_SMD:C_0402_1005Metric
- C8: renamed from C2; footprint (none) -> Capacitor_SMD:C_0805_2012Metric
- C9: renamed from C11; footprint (none) -> Capacitor_SMD:C_0805_2012Metric
- L1: value 1uH (1 ohm) -> FTC404030S1R0MGCA
- R1: renamed from R2; footprint (none) -> Resistor_SMD:R_0402_1005Metric
- R2: renamed from R3; footprint (none) -> Resistor_SMD:R_0402_1005Metric
- R3: renamed from R5; footprint (none) -> Resistor_SMD:R_0402_1005Metric
- U2: footprint (none) -> Package_DFN_QFN:TDFN-8-1EP_2x2mm_P0.5mm_EP0.8x1.2mm
- renumbered C5 to C11, C6 to C13, C7 to C14, C8 to C15, C3 to C16, C4 to C17, C9 to C18, C10 to C20, D9 to D1, D8 to D2, D7 to D3, D5 to D4, D2 to D5, D1 to D6, D4 to D7, D6 to D8, J3 to J1, J6 to J2, R1 to R4, R4 to R5, U4 to U3, U6 to U5, U9 to U6, U5 to U8, U3 to U9, X2 to X1
Connections:
- net +3V3: now also C19.1, U4.8 (VCC), U7.8 (VCC)
- net +BATT: now also SW2.2 (B); no longer J2.2 (Pin_2)
- net GND: now also C1.1, C19.2, U4.4 (GND), U7.4 (GND), U7.9 (EP)
- net SCL: now also U4.6 (SCL)
- net SDA: now also U4.5 (SDA)
- net at U1.20 (XIN), X1.1 (OSC1): now also C1.2
- net QSPI_SD3: now reaches U1.51 (QSPI_SD3)
- net QSPI_SD3: now also U7.7 (HOLD#orRESET#(IO3))
- net QSPI_SCLK: now reaches U1.52 (QSPI_SCLK)
- net QSPI_SCLK: now also U7.6 (CLK)
- net QSPI_SD0: now reaches U1.53 (QSPI_SD0)
- net QSPI_SD0: now also U7.5 (DI(IO0))
- net QSPI_SD2: now reaches U1.54 (QSPI_SD2)
- net QSPI_SD2: now also U7.3 (WP#(IO2))
- net QSPI_SD1: now reaches U1.55 (QSPI_SD1)
- net QSPI_SD1: now also U7.2 (DO(IO1))
- net ~{QSPI_SS}: now reaches U1.56 (~{QSPI_SS})
- net ~{QSPI_SS}: now also U7.1 (CS#)
- new net: J2.2 (Pin_2), SW2.1 (A)
- new net WP: U4.7 (WP)
- no-connect marks 10 -> 15
Other:
- note added: "LoRa connector"
- note added: "Program flash"
- note added: "Storage flash"
- note removed: "LORA Connector"
- note removed: "Storage Flash"
- moved on the sheet: C2, CN2, D1, D2, D3, D4, J2, X1
