File: Lora/loracircle/loracircle.kicad_sch (KiCad schematic)
At the start: 12 parts, among them U1 RFM69HCW, U3 AP2112K-3.3, X1 uFL/SMA

Commit message: Lora sch done
Parts:
- removed JP1: HEADER-1X570MIL, Adafruit RFM+LoRa Breakout:1X05_ROUND_70, symbol Adafruit RFM+LoRa Breakout-eagle-import:HEADER-1X570MIL
- removed R1: 100K, Adafruit RFM+LoRa Breakout:0805-NO, symbol Adafruit RFM+LoRa Breakout-eagle-import:RESISTOR0805_NOOUTLINE
- removed U3: AP2112K-3.3, Adafruit RFM+LoRa Breakout:SOT23-5, symbol Adafruit RFM+LoRa Breakout-eagle-import:VREG_SOT23-5
Connections:
- net VIN is gone; now on net 3.3V: C3.1, JP3.1, R2.2, R3.2
- net DIO1: no longer names the net of U1.7P (DIO1)
- net DIO2: no longer names the net of U1.8P (DIO2)
- net DIO3: no longer names the net of U1.3P (DIO3)
- net DIO4: no longer names the net of U1.4P (DIO4)
- net DIO5: no longer names the net of U1.15P (DIO5)
Other:
- moved on the sheet: C2, C3

Commit message: DESC
Just transferring files from school computer
Parts:
- removed JP2: HEADER-1X1ROUND, Adafruit RFM+LoRa Breakout:1X01_ROUND, symbol Adafruit RFM+LoRa Breakout-eagle-import:HEADER-1X1ROUND
- removed X1: uFL/SMA, Adafruit RFM+LoRa Breakout:SMA_EDGELAUNCH_UFL, symbol Adafruit RFM+LoRa Breakout-eagle-import:SMACONNECTOR_EDGE_UFL
- added J1: CONMHF1-SMD-T, CONMHF1-SMD-T:TE_CONMHF1-SMD-T, symbol CONMHF1-SMD-T:CONMHF1-SMD-T
- C1, C2, C3, R2, R3: footprint Adafruit RFM+LoRa Breakout:0805-NO -> LIBRARY:0805-NO
- JP3: footprint Adafruit RFM+LoRa Breakout:1X09_ROUND_70 -> LIBRARY:CONN_B9B-PH-SM4-TB_JST
- U1: footprint Adafruit RFM+LoRa Breakout:RFMHCW_SMT -> LIBRARY:RFMHCW_SMT
Connections:
- net GND: now also J1.2, J1.3, J1.4
- net at U1.1P (ANT): now also J1.1

Commit message: prettify lora board
Parts:
- C1, C3: footprint LIBRARY:0805-NO -> Capacitor_SMD:C_0805_2012Metric
- C2: footprint LIBRARY:0805-NO -> Capacitor_SMD:C_0603_1608Metric
- JP3: footprint LIBRARY:CONN_B9B-PH-SM4-TB_JST -> Connector_JST:JST_PH_B9B-PH-SM4-TB_1x09-1MP_P2.00mm_Vertical
- R2, R3: footprint LIBRARY:0805-NO -> Resistor_SMD:R_0603_1608Metric
Changed lines of the file:
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@@
 			)
 		)
-		(property "Footprint" "LIBRARY:0805-NO"
+		(property "Footprint" "Capacitor_SMD:C_0603_1608Metric"
 			(at 143.51 55.88 0)
 			(hide yes)
@@
 			)
 		)
-		(property "Footprint" "LIBRARY:0805-NO"
+		(property "Footprint" "Capacitor_SMD:C_0805_2012Metric"
 			(at 190.5 97.79 0)
 			(hide yes)
@@
 			)
 		)
-		(property "Footprint" "LIBRARY:CONN_B9B-PH-SM4-TB_JST"
+		(property "Footprint" "Connector_JST:JST_PH_B9B-PH-SM4-TB_1x09-1MP_P2.00mm_Vertical"
 			(at 238.76 72.39 0)
 			(hide yes)
@@
 			)
 		)
-		(property "Footprint" "LIBRARY:0805-NO"
+		(property "Footprint" "Resistor_SMD:R_0603_1608Metric"
 			(at 205.74 67.31 0)
 			(hide yes)
@@
 			)
 		)
-		(property "Footprint" "LIBRARY:0805-NO"
+		(property "Footprint" "Capacitor_SMD:C_0805_2012Metric"
 			(at 152.4 55.88 0)
 			(hide yes)
@@
 			)
 		)
-		(property "Footprint" "LIBRARY:0805-NO"
+		(property "Footprint" "Resistor_SMD:R_0603_1608Metric"
 			(at 198.12 67.31 0)
 			(hide yes)
