File: KiCad/Fireball FC/fireball_fc/fireball_fc.kicad_pcb (KiCad board)
At the start: 2 copper layers, 74 x 60.5 mm, 34 parts, among them CN1 HDGC2001WR-S-4P, CN2 HDGC2001WR-S-3P, J3 Conn_01x04, J6 Conn_01x02, P1 USB_C_Plug_USB2.0, SW1 HX 3X4X2-2P-2.5N-04, U1 RP2040, U3 MS5607-02BA, U4 TPS61023, U5 LSM6DSO, U6 NCP708, U7 W25Q128JVS, U8 W25Q16JVUXIQ, U9 HDGC2001WR-S-9P, X2 12MHZ Crystal

Commit message: added inductor. Will do other stuff soon
Parts:
- added L2: FTC404030S1R0MGCA, lcsc_footprints:C39676079_IND-SMD_L4_1-W4_1_SPM40XX, F.Cu at (230.7, 120.0)
- added U7: W25Q16JVUXIQ, lcsc_footprints:C2843335_USON-8_L3_0-W2_0-P0_50-BL-EP, F.Cu at (235.1, 119.6)
- renumbered C5 to C11, C6 to C13, C7 to C14, C8 to C15, C3 to C16, C4 to C17, C9 to C18, C10 to C20, D9 to D1, D8 to D2, D7 to D3, D5 to D4, D2 to D5, D1 to D6, D4 to D7, D6 to D8, J3 to J1, J6 to J2, CN2 to J3, U9 to J4, CN1 to J5, R1 to R4, R4 to R5, U4 to U3, U6 to U5, U5 to U8, U3 to U9, X2 to X1
Connections:
- J2 pad 2: +BATT -> Net-(J2-Pin_2)
- J4 pad 9: 3.3V -> +3V3
- P1 pad A5: unconnected-(P1-CC-PadA5) -> Net-(P1-CC)
- U1 pad 19: unconnected-(U1-TESTEN-Pad19) -> GND
- U1 pad 43: unconnected-(U1-ADC_AVDD-Pad43) -> +3V3
- U1 pad 44: unconnected-(U1-VREG_VIN-Pad44) -> +3V3
- U1 pad 48: unconnected-(U1-USB_VDD-Pad48) -> +3V3
- U1 pad 51: Net-(U1-QSPI_SD3) -> /QSPI_SD3
- U1 pad 52: Net-(U1-QSPI_SCLK) -> /QSPI_SCLK
- U1 pad 53: Net-(U1-QSPI_SD0) -> /QSPI_SD0
- U1 pad 54: Net-(U1-QSPI_SD2) -> /QSPI_SD2
- U1 pad 55: Net-(U1-QSPI_SD1) -> /QSPI_SD1
- U1 pad 56: Net-(U1-~{QSPI_SS}) -> /~{QSPI_SS}

Commit message: Description
-Added new USB that had the proper cc lines broken out
-Wired all modules
-added i2c pull up
-added logos for silkscreen
-drank a watermelon poppi!!
-added resistors on the usb
-added bootsel button
Parts:
- added G***: LOGO, lcsc_footprints:issaclogo, F.Cu at (241.2, 73.5)
- added G***: LOGO, LOGO, F.Cu at (247.2, 74.2)
- added USB1: USB-TYPE-C-020, lcsc_footprints:C2927040_USB-SMD_USB-TYPE-C-020, F.Cu at (247.2, 136.9)
Connections:
- SW1 pad 1: unconnected-(SW1-Pad1) -> GND
- SW1 pad 2: unconnected-(SW1-Pad2) -> Net-(R6-Pad2)
- U1 pad 11: unconnected-(U1-GPIO8-Pad11) -> /SDA
- U1 pad 12: unconnected-(U1-GPIO9-Pad12) -> /SCL
- U1 pad 15: unconnected-(U1-GPIO12-Pad15) -> /GPS_RX
- U1 pad 16: unconnected-(U1-GPIO13-Pad16) -> /GPS_TX
- U1 pad 17: unconnected-(U1-GPIO14-Pad17) -> /NEOPIXEL
- U1 pad 18: unconnected-(U1-GPIO15-Pad18) -> /BUZZER
- U1 pad 26: unconnected-(U1-RUN-Pad26) -> Net-(U1-RUN)
- U1 pad 27: unconnected-(U1-GPIO16-Pad27) -> /SDLED
