File: KiCad/Fireball FC/fireball_fc/fireball_fc.kicad_sch (KiCad schematic)
At the start: 53 parts, among them CN1 HDGC2001WR-S-4P, CN2 HDGC2001WR-S-3P, J1 Conn_01x04, J2 Conn_01x02, P1 USB_C_Plug_USB2.0, SW1 HX 3X4X2-2P-2.5N-04, SW2 MAIN POWER, U1 RP2040, U2 MAX17048G, U3 TPS61023, U4 CAT24C256WI-GT3, U5 NCP708, U6 HDGC2001WR-S-9P, U7 W25Q16JVUXIQ, U8 LSM6DSO, U9 MS5607-02BA, X1 12MHZ Crystal

Commit message: organize some things
Parts:
- renumbered CN2 to J3, U6 to J4, CN1 to J5
Connections:
- net +3V3: now also J4.9
- net 3.3V: no longer J4.9
- net BUZZER: now reaches BZ1.1 (+)
Other:
- moved on the sheet: C12, C19, J3, P1, R3, U7

Commit message: added inductor. Will do other stuff soon
Parts:
- removed L1: FTC404030S1R0MGCA, symbol Device:L_Small
- added L2: FTC404030S1R0MGCA, lcsc_footprints:C39676079_IND-SMD_L4_1-W4_1_SPM40XX, symbol lcsc_imported:FTC404030S1R0MGCA
Connections:
- net +BATT: now also L2.1
- net at U3.5 (SW): now also L2.2
Changed lines of the file:
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@@
 	)
 	(junction
-		(at 220.98 80.01)
-		(diameter 0)
-		(color 0 0 0 0)
-	)
-	(junction
 		(at 241.3 87.63)
 		(diameter 0)
@@
 	)
 	(junction
+		(at 220.98 80.01)
+		(diameter 0)
+		(color 0 0 0 0)
+	)
+	(junction
 		(at 355.6 76.2)
 		(diameter 0)
@@
 	(wire
 		(pts
+			(xy 231.14 78.74) (xy 231.14 80.01)
+		)
+		(stroke
+			(width 0)
+			(type default)
+		)
+	)
+	(wire
+		(pts
 			(xy 255.27 52.07) (xy 256.54 52.07)
 		)
@@
 	(wire
 		(pts
+			(xy 220.98 78.74) (xy 220.98 80.01)
+		)
+		(stroke
+			(width 0)
+			(type default)
+		)
+	)
+	(wire
+		(pts
 			(xy 382.27 213.36) (xy 386.08 213.36)
 		)
@@
 	(wire
 		(pts
-			(xy 228.6 80.01) (xy 231.14 80.01)
-		)
-		(stroke
-			(width 0)
-			(type default)
-		)
-	)
-	(wire
-		(pts
 			(xy 391.16 187.96) (xy 387.35 187.96)
 		)
@@
 	(wire
 		(pts
-			(xy 220.98 80.01) (xy 223.52 80.01)
-		)
-		(stroke
-			(width 0)
-			(type default)
-		)
-	)
-	(wire
-		(pts
 			(xy 318.77 168.91) (xy 330.2 168.91)
 		)
@@
 	)
 	(symbol
-		(lib_id "Device:L_Small")
-		(at 226.06 80.01 90)
-		(unit 1)
-		(body_style 1)
-		(exclude_from_sim no)
-		(in_bom yes)
-		(on_board yes)
-		(in_pos_files yes)
-		(dnp no)
-		(fields_autoplaced yes)
-		(property "Reference" "L1"
-			(at 226.06 74.93 90)
-			(show_name no)
-			(do_not_autoplace no)
-			(effects
-				(font
-					(size 1.27 1.27)
-				)
-			)
-		)
-		(property "Value" "FTC404030S1R0MGCA"
-			(at 226.06 77.47 90)
-			(show_name no)
-			(do_not_autoplace no)
-			(effects
-				(font
-					(size 1.27 1.27)
-				)
-			)
-		)
-		(property "Footprint" ""
-			(at 226.06 80.01 0)
-			(hide yes)
-			(show_name no)
-			(do_not_autoplace no)
-			(effects
-				(font
-					(size 1.27 1.27)
-				)
-			)
-		)
-		(property "Datasheet" ""
-			(at 226.06 80.01 0)
-			(hide yes)
-			(show_name no)
-			(do_not_autoplace no)
-			(effects
-				(font
-					(size 1.27 1.27)
-				)
-			)
-		)
-		(property "Description" "Inductor, small symbol"
-			(at 226.06 80.01 0)
-			(hide yes)
-			(show_name no)
-			(do_not_autoplace no)
-			(effects
-				(font
-					(size 1.27 1.27)
-				)
-			)
-		)
-		(pin "2"
-		)
-		(pin "1"
-		)
-		(instances
-			(project "fireball_fc"
-				(path "/a582df85-54b5-4502-ad28-1762afa22b26"
-					(reference "L1")
-					(unit 1)
-				)
-			)
-		)
-	)
-	(symbol
 		(lib_id "Switch:SW_SPST")
 		(at 320.04 124.46 0)
@@
 					(unit 1)
 				)
+			)
+		)
+	)
+	(symbol
+		(lib_id "lcsc_imported:FTC404030S1R0MGCA")
+		(at 226.06 78.74 0)
+		(unit 1)
+		(body_style 1)
+		(exclude_from_sim no)
+		(in_bom yes)
+		(on_board yes)
+		(in_pos_files yes)
+		(dnp no)
+		(fields_autoplaced yes)
+		(property "Reference" "L2"
+			(at 226.06 72.39 0)
+			(show_name no)
+			(do_not_autoplace no)
+			(effects
+				(font
+					(size 1.27 1.27)
+				)
+			)
+		)
+		(property "Value" "FTC404030S1R0MGCA"
+			(at 226.06 74.93 0)
+			(show_name no)
+			(do_not_autoplace no)
+			(effects
+				(font
+					(size 1.27 1.27)
+				)
+			)
+		)
+		(property "Footprint" "lcsc_footprints:C39676079_IND-SMD_L4_1-W4_1_SPM40XX"
+			(at 226.06 88.9 0)
+			(hide yes)
+			(show_name no)
+			(do_not_autoplace no)
+			(effects
+				(font
+					(size 1.27 1.27)
+				)
+			)
+		)
+		(property "Datasheet" "https://www.lcsc.com/datasheet/lcsc_datasheet_2409180941_cjiang--Changjiang-Microelectronics-Tech-FTC404030S1R0MGCA_C39676079.pdf"
+			(at 223.774 78.613 0)
+			(hide yes)
+			(show_name no)
+			(do_not_autoplace no)
+			(effects
+				(font
+					(size 1.27 1.27)
+				)
+			)
+		)
+		(property "Description" "FTC404030S1R0MGCA"
+			(at 226.06 78.74 0)
+			(hide yes)
+			(show_name no)
+			(do_not_autoplace no)
+			(effects
+				(font
+					(size 1.27 1.27)
+				)
+			)
+		)
+		(property "LCSC" "C39676079"
+			(at 226.06 78.74 0)
+			(hide yes)
+			(show_name no)
+			(do_not_autoplace no)
+			(effects
+				(font
+					(size 1.27 1.27)
+				)
+			)
+		)
+		(property "Manufacturer" "cjiang(长江微电)"
+			(at 226.06 78.74 0)
+			(hide yes)
+			(show_name no)
+			(do_not_autoplace no)
+			(effects
+				(font
+					(size 1.27 1.27)
+				)
+			)
+		)
+		(pin "1"
+		)
+		(pin "2"
+		)
+		(instances
+			(project "fireball_fc"
+				(path "/a582df85-54b5-4502-ad28-1762afa22b26"
+					(reference "L2")
+					(unit 1)
+				)

Commit message: Description
-Added new USB that had the proper cc lines broken out
-Wired all modules
-added i2c pull up
-added logos for silkscreen
-drank a watermelon poppi!!
-added resistors on the usb
-added bootsel button
Parts:
- removed P1: USB_C_Plug_USB2.0, Connector_USB:USB_C_Receptacle_GCT_USB4105-xx-A_16P_TopMnt_Horizontal, symbol Connector:USB_C_Plug_USB2.0
- added C21: 0.1uF, Capacitor_SMD:C_0805_2012Metric, symbol Device:C_Small
- added C22: 10uF, Capacitor_SMD:C_0805_2012Metric, symbol Device:C_Small
- added R10: maybebridgethis, Resistor_SMD:R_0402_1005Metric, symbol Device:R_Small
- added R11: 5.1k, Resistor_SMD:R_0402_1005Metric, symbol Device:R_Small
- added R6: 1K, Resistor_SMD:R_0402_1005Metric, symbol Device:R_Small
- added R7: NOFIT, Resistor_SMD:R_0402_1005Metric, symbol Device:R_Small
- added R8, R9: 4.7k, Resistor_SMD:R_0402_1005Metric, symbol Device:R_Small
- added USB1: USB-TYPE-C-020, lcsc_footprints:C2927040_USB-SMD_USB-TYPE-C-020, symbol lcsc_imported:USB-TYPE-C-020
Connections:
- net LORA_MISO is gone; now on net SPI0_MISO: J4.4
- net LORA_MOSI is gone; now on net SPI0_MOSI: J4.3
- net LORA_SCK is gone; now on net SPI0_SCK: J4.5
- net +3V3: now also Card1.4 (VDD), C21.2, C22.2, R10.2, R7.2, R8.2, R9.2
- net +5V: now also USB1.A4 (VBUS), USB1.A9 (VBUS), USB1.B4 (VBUS), USB1.B9 (VBUS)
- net 5V_EN: now also U1.32 (GPIO21)
- net BUZZER: now also U1.18 (GPIO15)
- net DVR: now also U1.34 (GPIO22)
- net GND: now also Card1.6 (VSS), SW1.1, C21.1, C22.1, R11.2, USB1.17 (SHELL), USB1.18 (SHELL), USB1.19 (SHELL), USB1.20 (SHELL), USB1.A1 (GND), USB1.A12 (GND), USB1.B1 (GND), USB1.B12 (GND)
- net GPS_RX: now also U1.15 (GPIO12)
- net GPS_TX: now also U1.16 (GPIO13)
- net LORA_CS: now also U1.8 (GPIO6)
- net LORA_DIO0: now also U1.9 (GPIO7)
- net LORA_EN: now also U1.14 (GPIO11)
- net LORA_RST: now also U1.13 (GPIO10)
- net NEOPIXEL: now also U1.17 (GPIO14)
- net SCL: now also U1.12 (GPIO9), R9.1
- net SDA: now also U1.11 (GPIO8), R8.1
- net SDLED: now also U1.27 (GPIO16)
- net USBDATA+: now also USB1.A6 (Dp1), USB1.B6 (Dp2)
- net USBDATA-: now also USB1.A7 (Dn1), USB1.B7 (Dn2)
- net ~{QSPI_SS}: now also R6.1, R7.1
- net at R3.2: now also USB1.A5 (CC1)
- net SD_CS: now reaches Card1.2 (CD/DAT3)
- net SD_CS: now also U1.7 (GPIO5)
- net SPI0_MOSI: now reaches Card1.3 (CMD)
- net SPI0_MOSI: now also U1.5 (GPIO3)
- net SPI0_SCK: now reaches Card1.5 (CLK)
- net SPI0_SCK: now also U1.4 (GPIO2)
- net SPI0_MISO: now reaches Card1.7 (DAT0)
- net SPI0_MISO: now also U1.6 (GPIO4)
- net at U1.26 (RUN): now also R10.1
- net at SW1.2: now also R6.2
- new net: R11.1, USB1.B5 (CC2)
- no-connect marks 15 -> 19
Other:
- note added: "---->"
- note added: "I think this is Card Detection. I left it as NC"
- note added: "bootsel (force usb)"
- note added: "hi"
- note added: "i2c pullup"
- note removed: "use the one that I just imported"
- moved on the sheet: C11, C13, C14, C15, Card1, D5, D6, R3, SW1, U5

Commit message: PCB Layout
Parts:
- removed BZ1: Buzzer, Buzzer_Beeper:Buzzer_CUI_CPT-9019S-SMT, symbol Device:Buzzer
- removed J2: Conn_01x02, Connector_PinSocket_2.54mm:PinSocket_1x02_P2.54mm_Vertical, symbol Connector_Generic:Conn_01x02
- added BUZ1: CPT-9019S-SMT-TR, lcsc_footprints:C95163_BUZ-SMD_L9_0-W9_0-P8_00-LS9_3, symbol lcsc_imported:CPT-9019S-SMT-TR
- added CN1: HDGC2001WR-S-2P, lcsc_footprints:C2936224_CONN-SMD_2P-P2_00_HDGC_HDGC2001WR-S-2P, symbol lcsc_imported:HDGC2001WR-S-2P
Connections:
- net BUZZER: now also BUZ1.1 (+)
- net GND: now also BUZ1.2 (-), CN1.1, CN1.3, CN1.4
- net at SW2.1 (A): now also CN1.2
Other:
- moved on the sheet: SW2
